File: Hardware/Qduino_Mini.sch (EAGLE design)
At the start: 43 parts, among them Q1 PFET, U1 ATMEGA32U41:1-LESS_PASTE, U2 MCP73831, U3 MAX17048, U4 TPS78233, U5 MIGHTYQ-L-SILK, U6 MIGHTYQ-S-SILK, U7 DNP, Y1 8MHZ

Commit message: testing out a reduced sized die pad to provide the recommended mechanical support, but with low pad to pin short likelihood
Parts:
- U1: value ATMEGA32U41:1-LESS_PASTE -> ATMEGA32U4QFN-44-PROD-OPTIMIZED; device SparkFun-DigitalIC:ATMEGA32U41:1-LESS_PASTE -> Testing:ATMEGA32U4QFN-44-PROD-OPTIMIZED
Changed lines of the file:
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@@
 <attribute name="PROD_ID" value="CONN-11443"/>
 </part>
-<part name="U1" library="SparkFun-DigitalIC" deviceset="ATMEGA32U4" device="1:1-LESS_PASTE" value="ATMEGA32U41:1-LESS_PASTE">
+<part name="U1" library="Testing" deviceset="ATMEGA32U4" device="QFN-44-PROD-OPTIMIZED" value="ATMEGA32U4QFN-44-PROD-OPTIMIZED">
 <attribute name="PROD_ID" value="IC-10828"/>
 </part>

Commit message: Used version of MCP73831 in current library, rather than legacy library. No real change.
Parts:
- U2: device SparkFun:MCP73831 -> SparkFun-PowerIC:MCP73831
Other:
- note added: "D"
- note added: "G"
- note added: "S"
Changed lines of the file:
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@@
 <part name="GND17" library="SparkFun" deviceset="GND" device=""/>
 <part name="GND18" library="SparkFun" deviceset="GND" device=""/>
-<part name="U2" library="SparkFun" deviceset="MCP73831" device="">
+<part name="U2" library="SparkFun-PowerIC" deviceset="MCP73831" device="">
 <attribute name="PROD_ID" value="IC-09995"/>
 </part>
@@
 <text x="41.91" y="-13.97" size="1.6764" layer="97">Can only run up to 13.3MHz @ 3V</text>
 <text x="62.23" y="-43.18" size="2.54" layer="94" ratio="5">Revised by: Brent Wilkins</text>
+<text x="130.048" y="45.72" size="1.778" layer="152" font="vector">D</text>
+<text x="130.302" y="55.118" size="1.778" layer="152" font="vector">S</text>
+<text x="125.73" y="51.562" size="1.778" layer="152" font="vector">G</text>
 </plain>
 <instances>

Commit message: Updated capactior ID
Parts:
- C1, C2: PROD_ID CAP-10300 -> CAP-08280
Changed lines of the file:
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@@
 </part>
 <part name="C2" library="SparkFun-Passives" deviceset="CAP" device="0603-CAP" value="4.7uF">
-<attribute name="PROD_ID" value="CAP-10300"/>
+<attribute name="PROD_ID" value="CAP-08280"/>
 </part>
 <part name="C1" library="SparkFun-Passives" deviceset="CAP" device="0603-CAP" value="4.7uF">
-<attribute name="PROD_ID" value="CAP-10300"/>
+<attribute name="PROD_ID" value="CAP-08280"/>
 </part>
 <part name="C4" library="SparkFun-Passives" deviceset="CAP" device="0603-CAP" value="1uF">
