File: Hardware/Qduino_Mini.sch (EAGLE design)
At the start: 43 parts, among them Q1 PFET, U1 ATMEGA32U41:1-LESS_PASTE, U2 MCP73831, U3 MAX17048, U4 TPS78233, U5 MIGHTYQ-L-SILK, U6 MIGHTYQ-S-SILK, U7 DNP, Y1 8MHZ

Commit message: Moved battery over to make rework easier.  In the process moved the power LED to the middle.  Also fixed RX/TX lines(D0/D1)
Parts:
- D1: value BAS16JTR -> 250mA/100V; device SparkFun-DiscreteSemi:DIODESOD -> SparkFun-DiscreteSemi:DIODEBAS16
- JP2: value USB_MICROB_PLUGCONN-11752 -> (none)
- LED1: value TX / YLW -> Yellow
- LED2: value RX / GRN -> GREEN
- LED3: value PWR / GRN -> GREEN
- LED4: value L / YLW -> Yellow
Connections:
- removed net RX: U1.PD2(RX), U7.TX
- removed net TX: U1.PD3(TX), U7.RX
- new net D0: U1.PD2(RX), U7.D0
- new net D1: U1.PD3(TX), U7.D1
Changed lines of the file:
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@@
 <layer number="113" name="IDFDebug" color="4" fill="1" visible="yes" active="yes"/>
 <layer number="116" name="Patch_BOT" color="9" fill="4" visible="no" active="yes"/>
+<layer number="118" name="Rect_Pads" color="7" fill="1" visible="yes" active="yes"/>
 <layer number="121" name="_tsilk" color="7" fill="1" visible="no" active="yes"/>
 <layer number="122" name="_bsilk" color="7" fill="1" visible="no" active="yes"/>
@@
 <part name="GND2" library="SFE Aesthetics" deviceset="GND" device=""/>
 <part name="GND3" library="SFE Aesthetics" deviceset="GND" device=""/>
-<part name="LED1" library="SparkFun-LED" deviceset="LED-YELLOW" device="0603" value="TX / YLW">
+<part name="LED1" library="SparkFun-LED" deviceset="LED-YELLOW" device="0603" value="Yellow">
 <attribute name="PROD_ID" value="DIO-09003"/>
 </part>
-<part name="LED2" library="SparkFun-LED" deviceset="LED-GREEN" device="0603" value="RX / GRN">
+<part name="LED2" library="SparkFun-LED" deviceset="LED-GREEN" device="0603" value="GREEN">
 <attribute name="PROD_ID" value="DIO-00821"/>
 </part>
 <part name="P+3" library="SFE Aesthetics" deviceset="VCC" device=""/>
-<part name="LED3" library="SparkFun-LED" deviceset="LED-GREEN" device="0603" value="PWR / GRN">
+<part name="LED3" library="SparkFun-LED" deviceset="LED-GREEN" device="0603" value="GREEN">
 <attribute name="PROD_ID" value="DIO-00821"/>
 </part>
 <part name="P+4" library="SFE Aesthetics" deviceset="VCC" device=""/>
 <part name="GND6" library="SFE Aesthetics" deviceset="GND" device=""/>
-<part name="LED4" library="SparkFun-LED" deviceset="LED-YELLOW" device="0603" value="L / YLW">
+<part name="LED4" library="SparkFun-LED" deviceset="LED-YELLOW" device="0603" value="Yellow">
 <attribute name="PROD_ID" value="DIO-09003"/>
 </part>
@@
 <part name="GND1" library="SparkFun" deviceset="GND" device=""/>
 <part name="GND9" library="SparkFun" deviceset="GND" device=""/>
-<part name="D1" library="SparkFun-DiscreteSemi" deviceset="DIODE" device="SOD" value="BAS16JTR"/>
+<part name="D1" library="SparkFun-DiscreteSemi" deviceset="DIODE" device="BAS16" value="250mA/100V"/>
 <part name="U5" library="SparkFun-Aesthetics" deviceset="MIGHTYQ-L-SILK" device=""/>
 <part name="U6" library="SparkFun-Aesthetics" deviceset="MIGHTYQ-S-SILK" device=""/>
@@
 </segment>
 </net>
-<net name="RX" class="0">
-<segment>
-<wire x1="-35.56" y1="88.9" x2="-38.1" y2="88.9" width="0.1524" layer="91"/>
-<pinref part="U1" gate="G$1" pin="PD2(RX)"/>
-<label x="-35.56" y="88.9" size="1.27" layer="95" xref="yes"/>
-</segment>
-<segment>
-<wire x1="-40.64" y1="2.54" x2="-38.1" y2="2.54" width="0.1524" layer="91"/>
-<pinref part="U7" gate="G$1" pin="TX"/>
-<label x="-38.1" y="2.54" size="1.27" layer="95" xref="yes"/>
-</segment>
-</net>
-<net name="TX" class="0">
-<segment>
-<wire x1="-35.56" y1="86.36" x2="-38.1" y2="86.36" width="0.1524" layer="91"/>
-<pinref part="U1" gate="G$1" pin="PD3(TX)"/>
-<label x="-35.56" y="86.36" size="1.27" layer="95" xref="yes"/>
-</segment>
-<segment>
-<wire x1="-40.64" y1="5.08" x2="-38.1" y2="5.08" width="0.1524" layer="91"/>
-<pinref part="U7" gate="G$1" pin="RX"/>
-<label x="-38.1" y="5.08" size="1.27" layer="95" xref="yes"/>
-</segment>
-</net>
 <net name="D4" class="0">
 <segment>
@@
 </segment>
 </net>
+<net name="D0" class="0">
+<segment>
+<pinref part="U7" gate="G$1" pin="D0"/>
+<wire x1="-40.64" y1="5.08" x2="-38.1" y2="5.08" width="0.1524" layer="91"/>
+<label x="-38.1" y="5.08" size="1.27" layer="95" xref="yes"/>
+</segment>
+<segment>
+<pinref part="U1" gate="G$1" pin="PD2(RX)"/>
+<wire x1="-38.1" y1="88.9" x2="-35.56" y2="88.9" width="0.1524" layer="91"/>
+<label x="-35.56" y="88.9" size="1.27" layer="95" xref="yes"/>
+</segment>
+</net>
+<net name="D1" class="0">
+<segment>
+<wire x1="-40.64" y1="2.54" x2="-38.1" y2="2.54" width="0.1524" layer="91"/>
+<pinref part="U7" gate="G$1" pin="D1"/>
+<label x="-38.1" y="2.54" size="1.27" layer="95" xref="yes"/>
+</segment>
+<segment>
+<wire x1="-35.56" y1="86.36" x2="-38.1" y2="86.36" width="0.1524" layer="91"/>
+<pinref part="U1" gate="G$1" pin="PD3(TX)"/>
+<label x="-35.56" y="86.36" size="1.27" layer="95" xref="yes"/>
+</segment>
+</net>
